File: sama5d27c_breakout.sch (KiCad schematic (older format))
At the start: 8 parts, among them J1 Conn_LCD, J2 Conn_JTAG, J3 Conn_SDMMC0, J4 Conn_FLEXCOM3_4, J5 Conn_DBGU, U1 SAMA5D2x-SIP

Commit message: Almost routed, just 2 unconnected left
Hahahahahah HahahaHhahaHAHAhahahHAHAHAHhahah
Parts:
- J1: footprint Connector_PinHeader_1.27mm:PinHeader_2x21_P1.27mm_Vertical -> Connector_PinHeader_1.27mm:PinHeader_2x19_P1.27mm_Vertical_SMD; symbol Connector_Generic:Conn_02x21_Odd_Even -> Connector_Generic:Conn_02x19_Odd_Even
Connections:
- net IRQ2: now also U1.B10 (PC27); no longer U1.H8 (PC25)
- net LCD_DAT0: now also J1.14 (Pin_14); no longer J1.18 (Pin_18)
- net LCD_DAT1: now also J1.15 (Pin_15); no longer J1.19 (Pin_19)
- net LCD_DAT10: now also J1.24 (Pin_24); no longer J1.28 (Pin_28)
- net LCD_DAT11: now also J1.25 (Pin_25); no longer J1.29 (Pin_29)
- net LCD_DAT12: now also J1.26 (Pin_26); no longer J1.30 (Pin_30)
- net LCD_DAT13: now also J1.27 (Pin_27); no longer J1.31 (Pin_31)
- net LCD_DAT14: now also J1.28 (Pin_28); no longer J1.32 (Pin_32)
- net LCD_DAT15: now also J1.29 (Pin_29); no longer J1.33 (Pin_33)
- net LCD_DAT16: now also J1.30 (Pin_30); no longer J1.34 (Pin_34)
- net LCD_DAT17: now also J1.31 (Pin_31); no longer J1.35 (Pin_35)
- net LCD_DAT18: now also J1.32 (Pin_32); no longer J1.36 (Pin_36)
- net LCD_DAT19: now also J1.33 (Pin_33); no longer J1.37 (Pin_37)
- net LCD_DAT2: now also J1.16 (Pin_16); no longer J1.20 (Pin_20)
- net LCD_DAT20: now also J1.34 (Pin_34); no longer J1.38 (Pin_38)
- net LCD_DAT21: now also J1.35 (Pin_35); no longer J1.39 (Pin_39)
- net LCD_DAT22: now also J1.36 (Pin_36); no longer J1.40 (Pin_40)
- net LCD_DAT23: now also J1.37 (Pin_37); no longer J1.41 (Pin_41)
- net LCD_DAT3: now also J1.17 (Pin_17); no longer J1.21 (Pin_21)
- net LCD_DAT4: now also J1.18 (Pin_18); no longer J1.22 (Pin_22)
- net LCD_DAT5: now also J1.19 (Pin_19); no longer J1.23 (Pin_23)
- net LCD_DAT6: now also J1.20 (Pin_20); no longer J1.24 (Pin_24)
- net LCD_DAT7: now also J1.21 (Pin_21); no longer J1.25 (Pin_25)
- net LCD_DAT8: now also J1.22 (Pin_22); no longer J1.26 (Pin_26)
- net LCD_DAT9: now also J1.23 (Pin_23); no longer J1.27 (Pin_27)
- net LCD_DEN: now also J1.10 (Pin_10); no longer J1.14 (Pin_14)
- net LCD_HSYNC: now also J1.11 (Pin_11); no longer J1.15 (Pin_15)
- net LCD_PCK: now also J1.13 (Pin_13); no longer J1.17 (Pin_17)
- net LCD_VSYNC: now also J1.12 (Pin_12); no longer J1.16 (Pin_16)
- net LED_BLUE: now also U1.F7 (PC26); no longer U1.P13 (PA31)
- net LED_GREEN: now also U1.G6 (PC16); no longer U1.F5 (PB0)
- net LED_RED: now also U1.H8 (PC25); no longer U1.R10 (PA10)
- net PMIC_CHGLEV: now also U1.L1 (PD16); no longer U1.N17 (PA12)
- net PMIC_LBO: now also U1.J2 (PD6); no longer U1.B2 (PC9)
- net USBB_PWR_EN: now also U1.K8 (PD15); no longer U1.R15 (PA27)
- net USR_BTN: now also U1.N1 (PD13); no longer U1.P14 (PA29)
- net SPI0_MISO: no longer names the net of U1.M11 (PA16)
- net SPI0_MISO: no longer J1.11 (Pin_11)
- net SPI0_MOSI: no longer names the net of U1.N16 (PA15)
- net SPI0_MOSI: no longer J1.12 (Pin_12)
- net SPI0_NPCS0: no longer names the net of U1.N14 (PA17)
- net SPI0_NPCS0: no longer J1.10 (Pin_10)
- net SPI0_SPCK: no longer names the net of U1.M17 (PA14)
- net SPI0_SPCK: no longer J1.13 (Pin_13)
- no-connect marks 34 -> 38
Other:
- note removed: "ETH_INT_IRQ_PD31"
- note removed: "GMDC_PD17"
- note removed: "GMDIO_PD18"
- note removed: "GRX0_PD13"
- note removed: "GRX1_PD14"
- note removed: "GRXDV_PD11"
- note removed: "GTX0_PD15"
- note removed: "GTX1_PD16"
- note removed: "GTXCK_PD09"
- note removed: "GTXEN_PD10"
- note removed: "PA23/FLEXCOM1_IO1/SPI1_MOSI/QSPI0_CS\n"
- note removed: "PA24/FLEXCOM1_IO0/SPI1_MISO/QSPI0_IO0\n"
- note removed: "PA25/FLEXCOM1_IO3/SPI1_NPCS0/QSPI0_IO1\n"
- note removed: "PA26/FLEXCOM1_IO4/SPI1_NPCS1/QSPI0_IO2\n"
- note removed: "PC11/ISI_D2/TCLK4/CANRX0/A0/NBS0\n"
- note removed: "PC12/ISI_D3/URXD3/TK0/A1\n"
- note removed: "PC13/ISI_D4/UTXD3/TF0/A2\n"
- note removed: "PC14/ISI_D5/TD0/A3\n"
- note removed: "PC15/ISI_D6/RD0/A4\n"
- note removed: "PC16/ISI_D7/RK0/A5\n"
- note removed: "PC17/ISI_D8/RF0/A6\n"
- note removed: "PC23/ISI_HSYNC/A12\n"
- note removed: "PC24/ISI_MCK/A13\n"
- note removed: "PC26/CANTX1/A15\n"
- note removed: "PC27/PCK1/CANRX1/A16\n"
- note removed: "PD06/PCK1/NCS2/PTCROW3\n"
- note removed: "PD07/NWR1/NBS1/PTCROW4\n"
- note removed: "PD08/NANDRDY/PTCROW5\n"
- note removed: "PD23/DBGU_RXD\n"
- note removed: "PD24/DBGU_TXD\n"
- note removed: "PD25/AD6\n"
- note removed: "PD26/AD7\n"
Changed lines of the file:
@@
 Wire Wire Line
 	3400 5200 3450 5200
-Text Notes 3500 4400 0    50   ~ 0
-PA23/FLEXCOM1_IO1/SPI1_MOSI/QSPI0_CS\n
-Text Notes 3500 4500 0    50   ~ 0
-PA24/FLEXCOM1_IO0/SPI1_MISO/QSPI0_IO0\n
-Text Notes 3500 4600 0    50   ~ 0
-PA25/FLEXCOM1_IO3/SPI1_NPCS0/QSPI0_IO1\n
-Text Notes 3500 4700 0    50   ~ 0
-PA26/FLEXCOM1_IO4/SPI1_NPCS1/QSPI0_IO2\n
 Wire Wire Line
 	6500 2100 6550 2100
@@
 Wire Wire Line
 	8850 5200 8900 5200
-Text Notes 8950 3200 0    50   ~ 0
-PC11/ISI_D2/TCLK4/CANRX0/A0/NBS0\n
-Text Notes 8950 3300 0    50   ~ 0
-PC12/ISI_D3/URXD3/TK0/A1\n
-Text Notes 8950 3400 0    50   ~ 0
-PC13/ISI_D4/UTXD3/TF0/A2\n
-Text Notes 8950 3500 0    50   ~ 0
-PC14/ISI_D5/TD0/A3\n
-Text Notes 8950 3600 0    50   ~ 0
-PC15/ISI_D6/RD0/A4\n
-Text Notes 8950 3700 0    50   ~ 0
-PC16/ISI_D7/RK0/A5\n
-Text Notes 8950 3800 0    50   ~ 0
-PC17/ISI_D8/RF0/A6\n
-Text Notes 8950 4400 0    50   ~ 0
-PC23/ISI_HSYNC/A12\n
-Text Notes 8950 4500 0    50   ~ 0
-PC24/ISI_MCK/A13\n
-Text Notes 8950 4700 0    50   ~ 0
-PC26/CANTX1/A15\n
-Text Notes 8950 4800 0    50   ~ 0
-PC27/PCK1/CANRX1/A16\n
 Wire Wire Line
 	11750 2100 11800 2100
@@
 Wire Wire Line
 	11750 5200 11800 5200
-Text Notes 11850 2700 0    50   ~ 0
-PD06/PCK1/NCS2/PTCROW3\n
-Text Notes 11850 2800 0    50   ~ 0
-PD07/NWR1/NBS1/PTCROW4\n
-Text Notes 11850 2900 0    50   ~ 0
-PD08/NANDRDY/PTCROW5\n
-Text Notes 11850 3000 0    50   ~ 0
-GTXCK_PD09
-Text Notes 11850 3100 0    50   ~ 0
-GTXEN_PD10
-Text Notes 11850 3200 0    50   ~ 0
-GRXDV_PD11
-Text Notes 11850 3300 0    50   ~ 0
-GRXDV_PD11
-Text Notes 11850 3400 0    50   ~ 0
-GRX0_PD13
-Text Notes 11850 3500 0    50   ~ 0
-GRX1_PD14
-Text Notes 11850 3600 0    50   ~ 0
-GTX0_PD15
-Text Notes 11850 3700 0    50   ~ 0
-GTX1_PD16
-Text Notes 11850 3800 0    50   ~ 0
-GMDC_PD17
-Text Notes 11850 3900 0    50   ~ 0
-GMDIO_PD18
-Text Notes 11850 4400 0    50   ~ 0
-PD23/DBGU_RXD\n
-Text Notes 11850 4500 0    50   ~ 0
-PD24/DBGU_TXD\n
-Text Notes 11850 4600 0    50   ~ 0
-PD25/AD6\n
-Text Notes 11850 4700 0    50   ~ 0
-PD26/AD7\n
 Text Label 6550 2600 0    50   ~ 0
 QSPI1_SCK
@@
 Text Label 6550 3100 0    50   ~ 0
 QSPI1_IO3
-Text Label 3450 3300 0    50   ~ 0
+Text Label 11800 3700 0    50   ~ 0
 PMIC_CHGLEV
 Text Label 3150 7000 2    50   ~ 0
@@
 Text Label 4300 6600 0    50   ~ 0
 PMIC_LBO
-Text Label 8900 3000 0    50   ~ 0
+Text Label 11800 2700 0    50   ~ 0
 PMIC_LBO
 Wire Wire Line
@@
 Text Label 7250 9350 2    50   ~ 0
 SDMMC0_DAT2
-Text Label 3450 5000 0    50   ~ 0
+Text Label 11800 3400 0    50   ~ 0
 USR_BTN
 Text Label 11800 4100 0    50   ~ 0
 USBA_VBUS_5V
-Text Label 3450 4800 0    50   ~ 0
+Text Label 11800 3600 0    50   ~ 0
 USBB_PWR_EN
 Text Label 11800 4000 0    50   ~ 0
 USBB_OVERCURR
-Text Label 3450 3100 0    50   ~ 0
+Text Label 8900 4600 0    50   ~ 0
 LED_RED
-Text Label 6550 2100 0    50   ~ 0
+Text Label 8900 3700 0    50   ~ 0
 LED_GREEN
-Text Label 3450 5200 0    50   ~ 0
+Text Label 8900 4700 0    50   ~ 0
 LED_BLUE
 Text Label 7250 6650 2    50   ~ 0
@@
 LCD_DISP
 Text Label 7850 6950 0    50   ~ 0
-SPI0_NPCS0
+LCD_DEN
 Text Label 7250 7050 2    50   ~ 0
-SPI0_MISO
+LCD_HSYNC
 Text Label 7850 7050 0    50   ~ 0
-SPI0_MOSI
+LCD_VSYNC
 Text Label 7250 7150 2    50   ~ 0
-SPI0_SPCK
+LCD_PCK
 Text Label 7850 7150 0    50   ~ 0
-LCD_DEN
+LCD_DAT0
 Text Label 7250 7250 2    50   ~ 0
-LCD_HSYNC
+LCD_DAT1
 Text Label 7850 7250 0    50   ~ 0
-LCD_VSYNC
+LCD_DAT2
 Text Label 7250 7350 2    50   ~ 0
-LCD_PCK
+LCD_DAT3
 Text Label 7850 7350 0    50   ~ 0
-LCD_DAT0
+LCD_DAT4
 Text Label 7250 7450 2    50   ~ 0
-LCD_DAT1
+LCD_DAT5
 Text Label 7850 7450 0    50   ~ 0
-LCD_DAT2
+LCD_DAT6
 Text Label 7250 7550 2    50   ~ 0
-LCD_DAT3
+LCD_DAT7
 Text Label 7850 7550 0    50   ~ 0
-LCD_DAT4
+LCD_DAT8
 Text Label 7250 7650 2    50   ~ 0
-LCD_DAT5
+LCD_DAT9
 Text Label 7850 7650 0    50   ~ 0
-LCD_DAT6
+LCD_DAT10
 Text Label 7250 7750 2    50   ~ 0
-LCD_DAT7
+LCD_DAT11
 Text Label 7850 7750 0    50   ~ 0
-LCD_DAT8
+LCD_DAT12
 Text Label 7250 7850 2    50   ~ 0
-LCD_DAT9
+LCD_DAT13
 Text Label 7850 7850 0    50   ~ 0
-LCD_DAT10
+LCD_DAT14
 Text Label 7250 7950 2    50   ~ 0
-LCD_DAT11
+LCD_DAT15
 Text Label 7850 7950 0    50   ~ 0
-LCD_DAT12
+LCD_DAT16
 Text Label 7250 8050 2    50   ~ 0
-LCD_DAT13
+LCD_DAT17
 Text Label 7850 8050 0    50   ~ 0
-LCD_DAT14
+LCD_DAT18
 Text Label 7250 8150 2    50   ~ 0
-LCD_DAT15
+LCD_DAT19
 Text Label 7850 8150 0    50   ~ 0
-LCD_DAT16
+LCD_DAT20
 Text Label 7250 8250 2    50   ~ 0
-LCD_DAT17
+LCD_DAT21
 Text Label 7850 8250 0    50   ~ 0
-LCD_DAT18
+LCD_DAT22
 Text Label 7250 8350 2    50   ~ 0
-LCD_DAT19
-Text Label 7850 8350 0    50   ~ 0
-LCD_DAT20
-Text Label 7250 8450 2    50   ~ 0
-LCD_DAT21
-Text Label 7850 8450 0    50   ~ 0
-LCD_DAT22
-Text Label 7250 8550 2    50   ~ 0
 LCD_DAT23
 $Comp
@@
 $EndComp
 $Comp
-L Connector_Generic:Conn_02x21_Odd_Even J1
+L Connector_Generic:Conn_02x19_Odd_Even J1
 U 1 1 5C8DA334
-P 7500 7550
-F 0 "J1" H 7550 8650 50  0000 C CNN
-F 1 "Conn_LCD" H 7550 6450 50  0000 C CNN
-F 2 "Connector_PinHeader_1.27mm:PinHeader_2x21_P1.27mm_Vertical" H 7500 7550 50  0001 C CNN
-F 3 "~" H 7500 7550 50  0001 C CNN
-	1    7500 7550
+P 7500 7450
+F 0 "J1" H 7550 8550 50  0000 C CNN
+F 1 "Conn_LCD" H 7550 6350 50  0000 C CNN
+F 2 "Connector_PinHeader_1.27mm:PinHeader_2x19_P1.27mm_Vertical_SMD" H 7500 7450 50  0001 C CNN
+F 3 "~" H 7500 7450 50  0001 C CNN
+	1    7500 7450
 	1    0    0    -1
 $EndComp
@@
 	7300 8350 7250 8350
 Wire Wire Line
-	7300 8450 7250 8450
-Wire Wire Line
-	7300 8550 7250 8550
-Wire Wire Line
 	7800 6550 7850 6550
 Wire Wire Line
@@
 Wire Wire Line
 	7800 8250 7850 8250
-Wire Wire Line
-	7800 8350 7850 8350
-Wire Wire Line
-	7800 8450 7850 8450
-NoConn ~ 7800 8550
+NoConn ~ 7800 8350
 Text Label 8900 2400 0    50   ~ 0
 LCD_PWM
-Text Label 8900 4600 0    50   ~ 0
+Text Label 8900 4800 0    50   ~ 0
 IRQ2
 Text Label 11800 2500 0    50   ~ 0
 LCD_TWD
-Text Label 3450 3800 0    50   ~ 0
-SPI0_NPCS0
-Text Label 3450 3600 0    50   ~ 0
-SPI0_MOSI
 Text Label 8900 2900 0    50   ~ 0
 LCD_DEN
@@
 Text Label 8900 2500 0    50   ~ 0
 LCD_DISP
-Text Label 3450 3700 0    50   ~ 0
-SPI0_MISO
-Text Label 3450 3500 0    50   ~ 0
-SPI0_SPCK
 Text Label 8900 2700 0    50   ~ 0
 LCD_HSYNC
@@
 	1    0    0    -1
 $EndComp
-NoConn ~ 11800 5200
-Text Notes 11850 5200 0    50   ~ 0
-ETH_INT_IRQ_PD31
 Text Label 8900 4900 0    50   ~ 0
 FLEXCOM4_IO0
@@
 Wire Wire Line
 	7800 10550 7850 10550
-NoConn ~ 3450 4400
-NoConn ~ 3450 4500
-NoConn ~ 3450 4600
-NoConn ~ 3450 4700
-NoConn ~ 8900 3200
-NoConn ~ 8900 3300
-NoConn ~ 8900 3400
-NoConn ~ 8900 3500
-NoConn ~ 8900 3600
-NoConn ~ 8900 3700
-NoConn ~ 8900 3800
-NoConn ~ 8900 4400
-NoConn ~ 8900 4500
-NoConn ~ 8900 4700
-NoConn ~ 8900 4800
-NoConn ~ 11800 4400
-NoConn ~ 11800 4500
-NoConn ~ 11800 4600
-NoConn ~ 11800 4700
-NoConn ~ 11800 2700
-NoConn ~ 11800 2800
-NoConn ~ 11800 2900
-NoConn ~ 11800 3000
-NoConn ~ 11800 3100
-NoConn ~ 11800 3200
-NoConn ~ 11800 3300
-NoConn ~ 11800 3400
-NoConn ~ 11800 3500
-NoConn ~ 11800 3600
-NoConn ~ 11800 3700
-NoConn ~ 11800 3800
-NoConn ~ 11800 3900
 Text Label 11800 2400 0    50   ~ 0
 DBGU_TX
@@
 F8 "USBB_D-" B R 3150 10500 50
 $EndSheet
+NoConn ~ 11800 5200
+NoConn ~ 11800 4400
+NoConn ~ 11800 4500
+NoConn ~ 11800 4600
+NoConn ~ 11800 4700
+NoConn ~ 11800 3500
+NoConn ~ 11800 3800
+NoConn ~ 11800 3900
+NoConn ~ 11800 2800
+NoConn ~ 11800 2900
+NoConn ~ 11800 3000
+NoConn ~ 11800 3100
+NoConn ~ 11800 3200
+NoConn ~ 11800 3300
+NoConn ~ 8900 3000
+NoConn ~ 6550 2100
+NoConn ~ 8900 3200
+NoConn ~ 8900 3300
+NoConn ~ 8900 3400
+NoConn ~ 8900 3500
+NoConn ~ 8900 3600
+NoConn ~ 8900 3800
+NoConn ~ 8900 4400
+NoConn ~ 8900 4500
+NoConn ~ 3450 3100
+NoConn ~ 3450 3300
+NoConn ~ 3450 3500
+NoConn ~ 3450 3600
+NoConn ~ 3450 3700
+NoConn ~ 3450 3800
+NoConn ~ 3450 4400
+NoConn ~ 3450 4500
+NoConn ~ 3450 4600
+NoConn ~ 3450 4700
+NoConn ~ 3450 4800
+NoConn ~ 3450 5000
+NoConn ~ 3450 5200
 $EndSCHEMATC
